File: pcb/casasagi_left/casasagi_left.kicad_pcb (KiCad board)
At the start: 2 copper layers, 133.3 x 82.7 mm, 114 parts, among them J101 USB_C_Receptacle_USB2.0, J102 AudioJack4, J103 Conn_01x05, SW101 RESET, SW102 BOOT, U101 TLV73333PDBV, U102 AT24CS32-XHM, U103 STM32F072C8Tx, Y101 8MHz

Commit message: add logo!!!!
Parts:
- added LOGO1: Casasagi_logo, casasagi:logo, B.Cu at (58.5, 82.0)

Commit message: add combined pcb
Routing:
- net +5V: track 664.6 -> 663.8 mm, vias 5 -> 4
- net GND: vias 157 -> 156

Commit message: prepare pcb for BOM and add BOM left
Routing:
- net GND: vias 156 -> 157
Changed lines of the file:
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@@
     (thickness 1.6)
     (drawings 62)
-    (tracks 1123)
+    (tracks 1124)
     (zones 0)
     (modules 115)
@@
   )
   (setup
-    (last_trace_width 0.5)
+    (last_trace_width 0.25)
     (user_trace_width 0.5)
     (user_trace_width 1)
@@
     (tags "LQFP QFP")
     (attr smd)
-    (fp_text reference U103 (at 0 5.85 90) (layer B.SilkS)
+    (fp_text reference U103 (at 1.75 6 90) (layer B.SilkS)
       (effects (font (size 0.8 0.8) (thickness 0.12)) (justify mirror))
     )
@@
     (tags SOD-123)
     (attr smd)
-    (fp_text reference D111 (at 0 2 90) (layer B.SilkS)
+    (fp_text reference D111 (at -4.25 -0.25 90) (layer B.SilkS)
       (effects (font (size 0.8 0.8) (thickness 0.12)) (justify mirror))
     )
@@
     (tags "SMD SMT crystal")
     (attr smd)
-    (fp_text reference Y101 (at 0 2.45) (layer B.SilkS)
+    (fp_text reference Y101 (at -3.75 1.5) (layer B.SilkS)
       (effects (font (size 0.8 0.8) (thickness 0.12)) (justify mirror))
     )
@@
     (tags capacitor)
     (attr smd)
-    (fp_text reference C109 (at 0 1.43) (layer B.SilkS)
+    (fp_text reference C109 (at 1 -1.5) (layer B.SilkS)
       (effects (font (size 0.8 0.8) (thickness 0.12)) (justify mirror))
     )
@@
     (tags capacitor)
     (attr smd)
-    (fp_text reference C104 (at 0 1.43) (layer B.SilkS)
+    (fp_text reference C104 (at 0 -1.5) (layer B.SilkS)
       (effects (font (size 0.8 0.8) (thickness 0.12)) (justify mirror))
     )
@@
     (tags capacitor)
     (attr smd)
-    (fp_text reference C105 (at 0 1.43 90) (layer B.SilkS)
+    (fp_text reference C105 (at 1.275 -2.525 180) (layer B.SilkS)
       (effects (font (size 0.8 0.8) (thickness 0.12)) (justify mirror))
     )
@@
     )
   )
-  (gr_text "Casasagi Left PCB / Rev. Alpha" (at 167.5 42.5) (layer B.SilkS)
-    (effects (font (size 1 1) (thickness 0.15)) (justify left mirror))
+  (gr_text "Casasagi Left PCB / Rev. Alpha" (at 172.5 78.5 270) (layer B.SilkS)
+    (effects (font (size 1 1) (thickness 0.15)) (justify mirror))
   )
-  (gr_text "(c) 2020, SMKiJ Casasagi Contributors" (at 74.75 42.5) (layer B.SilkS)
-    (effects (font (size 1 1) (thickness 0.15)) (justify left mirror))
+  (gr_text "(c) 2020, SMKiJ Casasagi Contributors" (at 41.75 78.75 270) (layer B.SilkS)
+    (effects (font (size 1 1) (thickness 0.15)) (justify mirror))
   )
   (dimension 6.5 (width 0.15) (layer Cmts.User)
@@
   (via (at 172.75 55.25) (size 0.8) (drill 0.4) (layers F.Cu B.Cu) (net 2))
   (via (at 172.75 63.75) (size 0.8) (drill 0.4) (layers F.Cu B.Cu) (net 2))
-  (via (at 172.75 78.5) (size 0.8) (drill 0.4) (layers F.Cu B.Cu) (net 2))
+  (via (at 171.25 78.5) (size 0.8) (drill 0.4) (layers F.Cu B.Cu) (net 2))
   (via (at 172.75 93) (size 0.8) (drill 0.4) (layers F.Cu B.Cu) (net 2))
   (via (at 172.75 102.25) (size 0.8) (drill 0.4) (layers F.Cu B.Cu) (net 2))
@@
   (via (at 41.5 115.75) (size 0.8) (drill 0.4) (layers F.Cu B.Cu) (net 2))
   (via (at 41.5 102) (size 0.8) (drill 0.4) (layers F.Cu B.Cu) (net 2))
-  (via (at 41.5 93.25) (size 0.8) (drill 0.4) (layers F.Cu B.Cu) (net 2))
-  (via (at 41.5 78.5) (size 0.8) (drill 0.4) (layers F.Cu B.Cu) (net 2))
-  (via (at 41.75 64) (size 0.8) (drill 0.4) (layers F.Cu B.Cu) (net 2))
+  (via (at 43.5 93.25) (size 0.8) (drill 0.4) (layers F.Cu B.Cu) (net 2))
+  (via (at 43 78.5) (size 0.8) (drill 0.4) (layers F.Cu B.Cu) (net 2))
+  (via (at 42.75 64) (size 0.8) (drill 0.4) (layers F.Cu B.Cu) (net 2))
   (via (at 41.75 55) (size 0.8) (drill 0.4) (layers F.Cu B.Cu) (net 2))
   (via (at 59.5 77) (size 0.8) (drill 0.4) (layers F.Cu B.Cu) (net 2))
@@
   (segment (start 94.375 41.875) (end 94.25 42) (width 0.25) (layer B.Cu) (net 2))
   (via (at 66.25 57) (size 0.8) (drill 0.4) (layers F.Cu B.Cu) (net 2))
+  (via (at 135.75 49) (size 0.8) (drill 0.4) (layers F.Cu B.Cu) (net 2))
   (segment (start 109.55 41.65) (end 109.725 41.825) (width 0.5) (layer B.Cu) (net 3) (status 30))
   (segment (start 100.75 56.8375) (end 100.75 57.640702) (width 0.25) (layer B.Cu) (net 3) (status 10))

Commit message: Change boss thru hole to M2 thru hole
Introduce M2 thru hole to fix switch plate and PCB together using M2 screw. Spacer style boss can be placed at the edge cutout.
Other:
- outline, holes or cut-outs redrawn

Commit message: replace M2 holes to drill holes
Parts:
- added H1: M2, MountingHole:MountingHole_2.2mm_M2, F.Cu at (59.5, 59.5)
- added H2: M2, MountingHole:MountingHole_2.2mm_M2, F.Cu at (59.5, 97.6)
- added H3: M2, MountingHole:MountingHole_2.2mm_M2, F.Cu at (154.8, 59.5)
- added H4: M2, MountingHole:MountingHole_2.2mm_M2, F.Cu at (154.8, 97.6)
- U102: value AT24CS32-XHM -> AT24C256C-XHL-T
Other:
- outline, holes or cut-outs redrawn
